File: PCBs/BME680_board/BME680.kicad_pcb (KiCad board)
At the start: 2 copper layers, 25.4 x 61 mm, 22 parts, among them J1 Conn_01x14, J2 Conn_01x14, J3 Conn_01x04, Q1 BC547, Q2 BC547, Q3 BC547, Q4 BC547, Q5 BC547

Commit message: added gerbers
Routing:
- net Earth: track 25.5 -> 55.1 mm
Changed lines of the file:
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@@
     (thickness 1.6)
     (drawings 5)
-    (tracks 114)
+    (tracks 125)
     (zones 0)
     (modules 22)
@@
   )
   (setup
-    (last_trace_width 0.7)
+    (last_trace_width 1.4)
     (user_trace_width 0.7)
     (user_trace_width 0.8)
     (user_trace_width 0.9)
     (user_trace_width 1)
+    (user_trace_width 1.4)
     (trace_clearance 0.2)
     (zone_clearance 0.508)
@@
     (visible_elements 7FFFFFFF)
     (pcbplotparams
-      (layerselection 0x010fc_ffffffff)
+      (layerselection 0x01000_fffffffe)
       (usegerberextensions false)
       (usegerberattributes false)
@@
       (outputformat 1)
       (mirror false)
-      (drillshape 1)
+      (drillshape 0)
       (scaleselection 1)
-      (outputdirectory ""))
+      (outputdirectory "../Gerber/BME680/"))
   )
   (net 0 "")
@@
   (gr_line (start 134.62 99.06) (end 134.62 134.62) (layer Edge.Cuts) (width 0.05))
   (segment (start 148.925409 124.124591) (end 148.971 124.079) (width 0.7) (layer B.Cu) (net 1))
-  (segment (start 148.938956 124.046956) (end 148.971 124.079) (width 0.7) (layer B.Cu) (net 1))
   (segment (start 144.399 100.993) (end 144.399 102.743) (width 1) (layer B.Cu) (net 1))
   (segment (start 146.459 98.933) (end 144.399 100.993) (width 1) (layer B.Cu) (net 1))
   (segment (start 155.829 98.933) (end 146.459 98.933) (width 1) (layer B.Cu) (net 1))
   (segment (start 146.196945 124.079) (end 146.164901 124.046956) (width 1) (layer B.Cu) (net 1))
-  (segment (start 148.971 124.079) (end 146.196945 124.079) (width 1) (layer B.Cu) (net 1))
   (segment (start 143.129 104.013) (end 144.399 102.743) (width 1) (layer B.Cu) (net 1))
   (segment (start 140.589 104.013) (end 143.129 104.013) (width 1) (layer B.Cu) (net 1))
   (segment (start 144.653 80.867) (end 144.685 80.899) (width 1) (layer B.Cu) (net 1))
   (segment (start 144.653 76.708) (end 144.653 80.867) (width 1) (layer B.Cu) (net 1))
-  (segment (start 152.019 109.093) (end 150.749 110.363) (width 1) (layer B.Cu) (net 2))
-  (segment (start 152.019 106.553) (end 152.019 109.093) (width 1) (layer B.Cu) (net 2))
+  (segment (start 148.938956 124.046956) (end 148.971 124.079) (width 1.4) (layer B.Cu) (net 1))
+  (segment (start 146.164901 124.046956) (end 148.938956 124.046956) (width 1.4) (layer B.Cu) (net 1))
+  (segment (start 144.685 80.899) (end 141.351 80.899) (width 1.4) (layer B.Cu) (net 1))
+  (segment (start 141.351 80.899) (end 136.398 85.852) (width 1.4) (layer B.Cu) (net 1))
+  (segment (start 136.398 85.852) (end 136.398 100.584) (width 1.4) (layer B.Cu) (net 1))
+  (segment (start 136.398 100.584) (end 137.16 100.584) (width 1.4) (layer B.Cu) (net 1))
+  (segment (start 137.16 100.584) (end 137.668 100.076) (width 1.4) (layer B.Cu) (net 1))
+  (segment (start 137.668 100.076) (end 137.668 98.298) (width 1.4) (layer B.Cu) (net 1))
+  (segment (start 137.668 98.298) (end 137.668 97.79) (width 1.4) (layer B.Cu) (net 1))
+  (segment (start 137.668 97.79) (end 137.16 97.282) (width 1.4) (layer B.Cu) (net 1))
   (segment (start 146.685 80.899) (end 151.511 80.899) (width 1) (layer B.Cu) (net 2))
   (segment (start 155.448 84.836) (end 155.448 85.471) (width 1) (layer B.Cu) (net 2))
@@
   (segment (start 146.685 80.899) (end 146.685 79.099) (width 1) (layer B.Cu) (net 2))
   (segment (start 146.685 79.099) (end 147.193 78.591) (width 1) (layer B.Cu) (net 2))
-  (segment (start 137.287 114.173) (end 140.589 114.173) (width 1) (layer B.Cu) (net 10))
+  (segment (start 150.90401 110.20799) (end 150.749 110.20799) (width 1.4) (layer B.Cu) (net 2))
+  (segment (start 152.019 109.093) (end 150.90401 110.20799) (width 1.4) (layer B.Cu) (net 2))
+  (segment (start 152.019 106.553) (end 152.019 109.093) (width 1.4) (layer B.Cu) (net 2))
+  (segment (start 140.589 114.173) (end 137.287 114.173) (width 1.4) (layer B.Cu) (net 10))
   (segment (start 150.622 122.682) (end 152.273 124.333) (width 0.7) (layer B.Cu) (net 14))
   (segment (start 149.733 116.967) (end 150.622 117.856) (width 0.7) (layer B.Cu) (net 14))
@@
   (segment (start 147.955 83.058) (end 146.05 83.058) (width 0.7) (layer B.Cu) (net 14))
   (segment (start 152.4 124.46) (end 152.273 124.333) (width 1) (layer B.Cu) (net 14))
-  (segment (start 152.4 128.651) (end 152.4 124.46) (width 1) (layer B.Cu) (net 14))
   (segment (start 140.589 98.933) (end 140.589 101.473) (width 1) (layer B.Cu) (net 14))
   (segment (start 137.287 106.553) (end 137.287 104.14) (width 1) (layer B.Cu) (net 14))
@@
   (segment (start 147.419 112.903) (end 149.733 115.217) (width 1) (layer B.Cu) (net 14))
   (segment (start 145.669 112.903) (end 147.419 112.903) (width 1) (layer B.Cu) (net 14))
+  (segment (start 152.273 128.524) (end 152.4 128.651) (width 1.4) (layer B.Cu) (net 14))
+  (segment (start 152.273 124.333) (end 152.273 128.524) (width 1.4) (layer B.Cu) (net 14))
   (segment (start 157.031081 106.553) (end 158.623 104.961081) (width 0.7) (layer B.Cu) (net 25))
   (segment (start 155.829 106.553) (end 157.031081 106.553) (width 0.7) (layer B.Cu) (net 25))
@@
   (segment (start 145.669 105.283) (end 145.669 102.743) (width 0.7) (layer B.Cu) (net 33))
   (segment (start 142.621 127.254) (end 142.621 108.331) (width 0.7) (layer B.Cu) (net 33))
-  (segment (start 147.32 128.651) (end 144.018 128.651) (width 1) (layer B.Cu) (net 33))
+  (segment (start 147.32 128.651) (end 144.018 128.651) (width 1.4) (layer B.Cu) (net 33))
   (segment (start 145.669 111.633) (end 146.144293 111.633) (width 0.7) (layer B.Cu) (net 34))
   (segment (start 145.923 114.935) (end 147.193 116.205) (width 0.7) (layer B.Cu) (net 34))
@@
   (segment (start 143.891 112.395) (end 143.891 113.919) (width 0.7) (layer B.Cu) (net 34))
   (segment (start 144.907 114.935) (end 145.923 114.935) (width 0.7) (layer B.Cu) (net 34))
-  (segment (start 147.193 117.221) (end 148.971 118.999) (width 1) (layer B.Cu) (net 34))
-  (segment (start 147.193 116.205) (end 147.193 117.221) (width 1) (layer B.Cu) (net 34))
+  (segment (start 147.193 117.221) (end 148.971 118.999) (width 1.4) (layer B.Cu) (net 34))
+  (segment (start 147.193 116.205) (end 147.193 117.221) (width 1.4) (layer B.Cu) (net 34))
   (segment (start 152.273 119.253) (end 152.273 116.205) (width 1) (layer B.Cu) (net 35))
-  (segment (start 152.273 114.427) (end 150.749 112.903) (width 1) (layer B.Cu) (net 35))
-  (segment (start 152.273 116.205) (end 152.273 114.427) (width 1) (layer B.Cu) (net 35))
+  (segment (start 152.273 114.427) (end 150.90401 113.05801) (width 1.4) (layer B.Cu) (net 35))
+  (segment (start 150.90401 113.05801) (end 150.749 113.05801) (width 1.4) (layer B.Cu) (net 35))
+  (segment (start 152.273 116.205) (end 152.273 114.427) (width 1.4) (layer B.Cu) (net 35))
 )
