File: PCBs/CU_board/CU/CU.sch (KiCad schematic (older format))
At the start: 48 parts, among them J1 Jack-DC, J10 Conn_01x04_Female, J11 Conn_01x04_Female, J12 Conn_01x04_Female, J13 Conn_01x15_Female, J14 Conn_01x15_Female, J2 Conn_01x04_Female, J3 Conn_01x04_Female, J4 Conn_01x04_Female, J5 Conn_01x04_Female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

Commit message: added gerbers
Connections:
- net at J9.7 (Pin_7): now also J9.8 (Pin_8)
Changed lines of the file:
@@
 Wire Wire Line
 	2700 4950 2700 5050
+Wire Wire Line
+	5350 4050 5300 4050
+Wire Wire Line
+	5300 4050 5300 4150
+Wire Wire Line
+	5300 4150 5350 4150
 $EndSCHEMATC
