File: PCBs/SenseBox_board/SB.sch (KiCad schematic (older format))
At the start: 13 parts, among them J1 Jack-DC, J2 Conn_01x20, J3 Conn_01x20, J7 Conn_01x08_Female, J9 Conn_01x08_Female

Commit message: added gerbers
Connections:
- net GND: now also J9.8 (Pin_8)
Changed lines of the file:
@@
 Wire Wire Line
 	3650 3150 3550 3150
+Wire Wire Line
+	6250 3900 6250 4000
+Wire Wire Line
+	6250 4000 6300 4000
 $EndSCHEMATC
