File: PCBs/TSL2561_board/TSL2561.kicad_pcb (KiCad board)
At the start: 2 copper layers, 25.4 x 51.4 mm, 22 parts, among them J1 Conn_01x05, J3 Conn_01x04, Q1 BC547, Q2 BC547, Q3 BC547, Q4 BC547, Q5 BC547

Commit message: added gerbers
Routing:
- net Earth: track 17.2 -> 32.2 mm
Changed lines of the file:
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@@
     (thickness 1.6)
     (drawings 5)
-    (tracks 107)
+    (tracks 118)
     (zones 0)
     (modules 22)
@@
     (visible_elements 7FFFFFFF)
     (pcbplotparams
-      (layerselection 0x010fc_ffffffff)
+      (layerselection 0x01000_fffffffe)
       (usegerberextensions false)
       (usegerberattributes false)
@@
       (outputformat 1)
       (mirror false)
-      (drillshape 1)
+      (drillshape 0)
       (scaleselection 1)
-      (outputdirectory ""))
+      (outputdirectory "../Gerber/TSL2561/"))
   )
   (net 0 "")
@@
   (segment (start 144.653 80.867) (end 144.685 80.899) (width 1) (layer B.Cu) (net 1))
   (segment (start 144.653 76.708) (end 144.653 80.867) (width 1) (layer B.Cu) (net 1))
-  (segment (start 149.479 117.602) (end 149.479 120.142) (width 1.4) (layer B.Cu) (net 16))
   (segment (start 138.43 106.68) (end 142.875 106.68) (width 1) (layer B.Cu) (net 1))
   (segment (start 146.69663 101.727) (end 148.68899 101.727) (width 1.4) (layer B.Cu) (net 1))
   (segment (start 142.875 106.68) (end 142.875 105.54863) (width 1.4) (layer B.Cu) (net 1))
   (segment (start 142.875 105.54863) (end 146.69663 101.727) (width 1.4) (layer B.Cu) (net 1))
+  (segment (start 144.685 80.899) (end 143.55363 80.899) (width 1.4) (layer B.Cu) (net 1))
+  (segment (start 143.55363 80.899) (end 140.716 80.899) (width 1.4) (layer B.Cu) (net 1))
+  (segment (start 140.716 80.899) (end 138.0236 83.5914) (width 1.4) (layer B.Cu) (net 1))
+  (segment (start 138.0236 83.5914) (end 138.0236 84.7598) (width 1.4) (layer B.Cu) (net 1))
+  (segment (start 138.0236 84.7598) (end 136.9568 85.8266) (width 1.4) (layer B.Cu) (net 1))
+  (segment (start 136.9568 85.8266) (end 136.2202 85.8266) (width 1.4) (layer B.Cu) (net 1))
+  (segment (start 136.2202 85.8266) (end 136.1948 85.8012) (width 1.4) (layer B.Cu) (net 1))
+  (segment (start 136.1948 85.8012) (end 136.1948 83.9724) (width 1.4) (layer B.Cu) (net 1))
+  (segment (start 136.1948 83.9724) (end 137.0584 83.9724) (width 1.4) (layer B.Cu) (net 1))
+  (segment (start 136.1948 83.9724) (end 136.2456 83.9724) (width 1.4) (layer B.Cu) (net 1))
+  (segment (start 136.2456 83.9724) (end 136.9822 84.709) (width 1.4) (layer B.Cu) (net 1))
   (segment (start 146.685 80.899) (end 151.511 80.899) (width 1) (layer B.Cu) (net 2))
   (segment (start 155.448 84.836) (end 155.448 85.471) (width 1) (layer B.Cu) (net 2))
@@
   (segment (start 158.115 97.79) (end 158.115 95.885) (width 1.4) (layer B.Cu) (net 2))
   (segment (start 158.115 102.235) (end 158.115 97.79) (width 1.4) (layer B.Cu) (net 2))
-  (segment (start 146.05 83.058) (end 143.637 85.471) (width 0.7) (layer B.Cu) (net 14))
-  (segment (start 150.368 85.471) (end 147.955 83.058) (width 0.7) (layer B.Cu) (net 14))
-  (segment (start 147.955 83.058) (end 146.05 83.058) (width 0.7) (layer B.Cu) (net 14))
-  (segment (start 152.908 85.471) (end 150.368 85.471) (width 1) (layer B.Cu) (net 14))
-  (segment (start 141.097 85.471) (end 143.637 85.471) (width 1) (layer B.Cu) (net 14))
   (segment (start 150.368 90.043) (end 151.638 91.313) (width 1) (layer B.Cu) (net 4))
   (segment (start 150.368 88.011) (end 150.368 90.043) (width 1) (layer B.Cu) (net 4))
@@
   (segment (start 150.114 101.727) (end 150.114 103.277) (width 0.8) (layer B.Cu) (net 11))
   (segment (start 150.114 103.277) (end 148.616 104.775) (width 0.8) (layer B.Cu) (net 11))
-  (segment (start 150.114 123.317) (end 149.479 122.682) (width 1.4) (layer B.Cu) (net 15))
-  (segment (start 154.559 123.317) (end 150.114 123.317) (width 1.4) (layer B.Cu) (net 15))
   (segment (start 149.733 107.95) (end 150.208293 107.95) (width 0.7) (layer B.Cu) (net 12))
   (segment (start 149.479 115.062) (end 149.479 112.522) (width 1.4) (layer B.Cu) (net 12))
@@
   (segment (start 154.559 112.522) (end 154.559 109.62901) (width 1.4) (layer B.Cu) (net 13))
   (segment (start 154.559 112.522) (end 154.559 115.57) (width 1.4) (layer B.Cu) (net 13))
+  (segment (start 146.05 83.058) (end 143.637 85.471) (width 0.7) (layer B.Cu) (net 14))
+  (segment (start 150.368 85.471) (end 147.955 83.058) (width 0.7) (layer B.Cu) (net 14))
+  (segment (start 147.955 83.058) (end 146.05 83.058) (width 0.7) (layer B.Cu) (net 14))
+  (segment (start 152.908 85.471) (end 150.368 85.471) (width 1) (layer B.Cu) (net 14))
+  (segment (start 141.097 85.471) (end 143.637 85.471) (width 1) (layer B.Cu) (net 14))
   (segment (start 154.559 120.777) (end 154.559 118.11) (width 1.4) (layer B.Cu) (net 14))
   (segment (start 151.765 116.44737) (end 151.765 110.871) (width 1) (layer B.Cu) (net 14))
@@
   (segment (start 140.815 108.585) (end 147.448 108.585) (width 0.9) (layer B.Cu) (net 14))
   (segment (start 138.43 109.22) (end 140.18 109.22) (width 0.9) (layer B.Cu) (net 14))
+  (segment (start 150.114 123.317) (end 149.479 122.682) (width 1.4) (layer B.Cu) (net 15))
+  (segment (start 154.559 123.317) (end 150.114 123.317) (width 1.4) (layer B.Cu) (net 15))
   (segment (start 140.97 114.173) (end 149.479 122.682) (width 0.9) (layer B.Cu) (net 15))
   (segment (start 146.05 110.62863) (end 145.27637 109.855) (width 0.9) (layer B.Cu) (net 15))
@@
   (segment (start 141.605 109.855) (end 140.97 110.49) (width 0.9) (layer B.Cu) (net 15))
   (segment (start 140.97 110.49) (end 140.97 114.173) (width 0.9) (layer B.Cu) (net 15))
+  (segment (start 149.479 117.602) (end 149.479 120.142) (width 1.4) (layer B.Cu) (net 16))
   (segment (start 148.717 117.602) (end 142.875 111.76) (width 1) (layer B.Cu) (net 16))
   (segment (start 149.479 117.602) (end 148.717 117.602) (width 1) (layer B.Cu) (net 16))
